Commit message: clean yumi URDF files, add to workcell, simstring and geometry functions

File: Fabrica/assets/yumi/yumi_left.urdf (robot description, URDF)
Before this commit: robot yumi, 9 links, 8 joints
Links:
- removed link yumi_link_1_l
- removed link yumi_link_2_l
- removed link yumi_link_3_l
- removed link yumi_link_4_l
- removed link yumi_link_5_l
- removed link yumi_link_6_l
- removed link yumi_link_7_l
- added link yumi_link_1, mass 2; collision mesh filename=collision/link_1.obj; visual mesh filename=visual/link_1.obj
- added link yumi_link_2, mass 2; collision mesh filename=collision/link_2.obj; visual mesh filename=visual/link_2.obj
- added link yumi_link_3, mass 2; collision mesh filename=collision/link_3.obj; visual mesh filename=visual/link_3.obj
- added link yumi_link_4, mass 2; collision mesh filename=collision/link_4.obj; visual mesh filename=visual/link_4.obj
- added link yumi_link_5, mass 2; collision mesh filename=collision/link_5.obj; visual mesh filename=visual/link_5.obj
- added link yumi_link_6, mass 2; collision mesh filename=collision/link_6.obj; visual mesh filename=visual/link_6.obj
- added link yumi_link_7, mass 2; collision mesh filename=collision/link_7.obj; visual mesh filename=visual/link_7.obj
Joints:
- removed joint yumi_joint_1_l
- removed joint yumi_joint_2_l
- removed joint yumi_joint_3_l
- removed joint yumi_joint_4_l
- removed joint yumi_joint_5_l
- removed joint yumi_joint_6_l
- removed joint yumi_joint_7_l
- added joint yumi_joint_1: type revolute, parent yumi_body, child yumi_link_1, origin xyz=0.05355 0.07250 0.41492 rpy=0.9781 -0.5716 2.3180, axis 0 0 1, limit lower=-2.94087978961 upper=2.94087978961 effort=300 velocity=3.14159265359
- added joint yumi_joint_2: type revolute, parent yumi_link_1, child yumi_link_2, origin xyz=0.03 0.0 0.1 rpy=1.57079632679 0.0 0.0, axis 0 0 1, limit lower=-2.50454747661 upper=0.759218224618 effort=300 velocity=3.14159265359
- added joint yumi_joint_3: type revolute, parent yumi_link_3, child yumi_link_4, origin xyz=-0.04188 0.0 0.07873 rpy=1.57079632679 -1.57079632679 0.0, axis 0 0 1, limit lower=-2.15548162621 upper=1.3962634016 effort=300 velocity=3.14159265359
- added joint yumi_joint_4: type revolute, parent yumi_link_4, child yumi_link_5, origin xyz=0.0405 0.16461 0.0 rpy=-1.57079632679 0.0 0.0, axis 0 0 1, limit lower=-5.06145483078 upper=5.06145483078 effort=300 velocity=6.98131700798
- added joint yumi_joint_5: type revolute, parent yumi_link_5, child yumi_link_6, origin xyz=-0.027 0 0.10039 rpy=1.57079632679 0.0 0.0, axis 0 0 1, limit lower=-1.53588974176 upper=2.40855436775 effort=300 velocity=6.98131700798
- added joint yumi_joint_6: type revolute, parent yumi_link_6, child yumi_link_7, origin xyz=0.027 0.029 0.0 rpy=-1.57079632679 0.0 0.0, axis 0 0 1, limit lower=-3.99680398707 upper=3.99680398707 effort=300 velocity=6.98131700798
- added joint yumi_joint_7: type revolute, parent yumi_link_2, child yumi_link_3, origin xyz=-0.03 0.17283 0.0 rpy=-1.57079632679 0.0 0.0, axis 0 0 1, limit lower=-2.94087978961 upper=2.94087978961 effort=300 velocity=3.14159265359

File: Fabrica/assets/yumi/yumi_right.urdf (robot description, URDF)
Before this commit: robot yumi, 9 links, 8 joints
Links:
- removed link yumi_link_1_r
- removed link yumi_link_2_r
- removed link yumi_link_3_r
- removed link yumi_link_4_r
- removed link yumi_link_5_r
- removed link yumi_link_6_r
- removed link yumi_link_7_r
- added link yumi_link_1, mass 2; collision mesh filename=collision/link_1.obj; visual mesh filename=visual/link_1.obj
- added link yumi_link_2, mass 2; collision mesh filename=collision/link_2.obj; visual mesh filename=visual/link_2.obj
- added link yumi_link_3, mass 2; collision mesh filename=collision/link_3.obj; visual mesh filename=visual/link_3.obj
- added link yumi_link_4, mass 2; collision mesh filename=collision/link_4.obj; visual mesh filename=visual/link_4.obj
- added link yumi_link_5, mass 2; collision mesh filename=collision/link_5.obj; visual mesh filename=visual/link_5.obj
- added link yumi_link_6, mass 2; collision mesh filename=collision/link_6.obj; visual mesh filename=visual/link_6.obj
- added link yumi_link_7, mass 2; collision mesh filename=collision/link_7.obj; visual mesh filename=visual/link_7.obj
Joints:
- removed joint yumi_joint_1_r
- removed joint yumi_joint_2_r
- removed joint yumi_joint_3_r
- removed joint yumi_joint_4_r
- removed joint yumi_joint_5_r
- removed joint yumi_joint_6_r
- removed joint yumi_joint_7_r
- added joint yumi_joint_1: type revolute, parent yumi_body, child yumi_link_1, origin xyz=0.05355 -0.0725 0.41492 rpy=-0.9795   -0.5682   -2.3155, axis 0 0 1, limit lower=-2.94087978961 upper=2.94087978961 effort=300 velocity=3.14159265359
- added joint yumi_joint_2: type revolute, parent yumi_link_1, child yumi_link_2, origin xyz=0.03 0.0 0.1 rpy=1.57079632679 0.0 0.0, axis 0 0 1, limit lower=-2.50454747661 upper=0.759218224618 effort=300 velocity=3.14159265359
- added joint yumi_joint_3: type revolute, parent yumi_link_3, child yumi_link_4, origin xyz=-0.04188 0.0 0.07873 rpy=1.57079632679 -1.57079632679 0.0, axis 0 0 1, limit lower=-2.15548162621 upper=1.3962634016 effort=300 velocity=3.14159265359
- added joint yumi_joint_4: type revolute, parent yumi_link_4, child yumi_link_5, origin xyz=0.0405 0.16461 0.0 rpy=-1.57079632679 0.0 0.0, axis 0 0 1, limit lower=-5.06145483078 upper=5.06145483078 effort=300 velocity=6.98131700798
- added joint yumi_joint_5: type revolute, parent yumi_link_5, child yumi_link_6, origin xyz=-0.027 0 0.10039 rpy=1.57079632679 0.0 0.0, axis 0 0 1, limit lower=-1.53588974176 upper=2.40855436775 effort=300 velocity=6.98131700798
- added joint yumi_joint_6: type revolute, parent yumi_link_6, child yumi_link_7, origin xyz=0.027 0.029 0.0 rpy=-1.57079632679 0.0 0.0, axis 0 0 1, limit lower=-3.99680398707 upper=3.99680398707 effort=300 velocity=6.98131700798
- added joint yumi_joint_7: type revolute, parent yumi_link_2, child yumi_link_3, origin xyz=-0.03 0.17283 0.0 rpy=-1.57079632679 0.0 0.0, axis 0 0 1, limit lower=-2.94087978961 upper=2.94087978961 effort=300 velocity=3.14159265359
